File: yo!macro/yo!macro.kicad_pcb (KiCad board)
At the start: 2 copper layers, 74.8 x 69.2 mm, 20 parts, among them J2 OLED, SW1 SW_Push, SW10 RotaryEncoder_Switch, SW11 SW_Push, SW12 SW_Push, SW13 SW_Push, SW14 SW_Push, SW2 SW_Push, SW3 SW_Push, SW4 RotaryEncoder_Switch, SW5 SW_Push, SW6 SW_Push, SW7 SW_Push, SW8 SW_Push, SW9 SW_Push, U1 ProMicro-kbd

Commit message: fix screen....
Parts:
- J2: moved to B.Cu
- moved J2 8.02 mm to (100.3, 127.2), turned to 180 degrees
Routing:
- net Switch14: track 33.4 -> 53.3 mm
- net vcc: track 32.9 -> 26.5 mm
- net Switch11: track 24.1 -> 24.8 mm, vias 0 -> 1
- net Switch12: track 23.4 -> 22.7 mm
